File: HW_Temperature_Sensors_Board/Espansione_NucleoH723ZG/Kicad_pj/H732_expansion.kicad_pcb (KiCad board)
At the start: 4 copper layers, 90.2 x 116.8 mm, 60 parts, among them CN1 CN11, CN2 CN8, CN3 CN9, CN4 CN7, CN5 CN10, CN6 C12, IC1 MAX31855TASA+, IC2 MAX490CSA+, IC3 CD4050BD, J1 Screw_Terminal_01x02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

Commit message: hw: connectors update
Other:
- board text added: "Morpho"
- board text added: "ZIO Connector"
Changed lines of the file:
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@@
     (pad "34" thru_hole oval (at 2.54 40.64 180) (size 1.7 1.7) (drill 1) (layers *.Cu *.Mask)
       (net 153 "unconnected-(CN5-Pad34)") (pinfunction "Pin_34") (pintype "passive+no_connect"))
-    (model "${KICAD6_3DMODEL_DIR}/Connector_PinHeader_2.54mm.3dshapes/PinHeader_2x17_P2.54mm_Vertical.wrl"
+    (model "${KICAD6_3DMODEL_DIR}/Connector_PinHeader_2.54mm.3dshapes/PinHeader_2x17_P2.54mm_Vertical.wrl" hide
       (offset (xyz 0 0 0))
       (scale (xyz 1 1 1))
@@
     (pad "16" thru_hole oval (at 2.54 17.78 180) (size 1.7 1.7) (drill 1) (layers *.Cu *.Mask)
       (net 253 "/connectors/MCU_to_ENC_CLK") (pinfunction "Pin_16") (pintype "passive"))
-    (model "${KICAD6_3DMODEL_DIR}/Connector_PinHeader_2.54mm.3dshapes/PinHeader_2x08_P2.54mm_Vertical.wrl"
+    (model "${KICAD6_3DMODEL_DIR}/Connector_PinHeader_2.54mm.3dshapes/PinHeader_2x08_P2.54mm_Vertical.wrl" hide
       (offset (xyz 0 0 0))
       (scale (xyz 1 1 1))
@@
     (pad "20" thru_hole oval (at 2.54 22.86 180) (size 1.7 1.7) (drill 1) (layers *.Cu *.Mask)
       (net 126 "unconnected-(CN4-Pad20)") (pinfunction "Pin_20") (pintype "passive+no_connect"))
-    (model "${KICAD6_3DMODEL_DIR}/Connector_PinHeader_2.54mm.3dshapes/PinHeader_2x10_P2.54mm_Vertical.wrl"
+    (model "${KICAD6_3DMODEL_DIR}/Connector_PinHeader_2.54mm.3dshapes/PinHeader_2x10_P2.54mm_Vertical.wrl" hide
       (offset (xyz 0 0 0))
       (scale (xyz 1 1 1))
@@
     (pad "30" thru_hole oval (at 2.54 35.56 180) (size 1.7 1.7) (drill 1) (layers *.Cu *.Mask)
       (net 107 "unconnected-(CN3-Pad30)") (pinfunction "Pin_30") (pintype "passive+no_connect"))
-    (model "${KICAD6_3DMODEL_DIR}/Connector_PinHeader_2.54mm.3dshapes/PinHeader_2x15_P2.54mm_Vertical.wrl"
+    (model "${KICAD6_3DMODEL_DIR}/Connector_PinHeader_2.54mm.3dshapes/PinHeader_2x15_P2.54mm_Vertical.wrl" hide
       (offset (xyz 0 0 0))
       (scale (xyz 1 1 1))
@@
     (pad "70" thru_hole oval (at 2.54 86.36 180) (size 1.7 1.7) (drill 1) (layers *.Cu *.Mask)
       (net 74 "unconnected-(CN1-Pad70)") (pinfunction "Pin_70") (pintype "passive+no_connect"))
-    (model "${KICAD6_3DMODEL_DIR}/Connector_PinHeader_2.54mm.3dshapes/PinHeader_2x35_P2.54mm_Vertical.wrl"
+    (model "${KICAD6_3DMODEL_DIR}/Connector_PinHeader_2.54mm.3dshapes/PinHeader_2x35_P2.54mm_Vertical.wrl" hide
       (offset (xyz 0 0 0))
       (scale (xyz 1 1 1))
@@
     (pad "70" thru_hole oval (at 2.54 86.36 180) (size 1.7 1.7) (drill 1) (layers *.Cu *.Mask)
       (net 223 "unconnected-(CN6-Pad70)") (pinfunction "Pin_70") (pintype "passive+no_connect"))
-    (model "${KICAD6_3DMODEL_DIR}/Connector_PinHeader_2.54mm.3dshapes/PinHeader_2x35_P2.54mm_Vertical.wrl"
+    (model "${KICAD6_3DMODEL_DIR}/Connector_PinHeader_2.54mm.3dshapes/PinHeader_2x35_P2.54mm_Vertical.wrl" hide
       (offset (xyz 0 0 0))
       (scale (xyz 1 1 1))
@@
     (effects (font (size 1.000759 1.000759) (thickness 0.14986)) (justify left))
   )
+  (gr_text "Morpho" (at 95.33 76.29) (layer "F.SilkS")
+    (effects (font (size 1.000759 1.000759) (thickness 0.25019)))
+  )
   (gr_text "Thermocouple T\n\n\n-250°C +400°C" (at 123.825 58.293 180) (layer "F.SilkS")
     (effects (font (size 1.000759 1.000759) (thickness 0.14986)))
@@
     (effects (font (size 1.000759 1.000759) (thickness 0.14986)))
   )
+  (gr_text "ZIO\nConnector" (at 102.83 95.5) (layer "F.SilkS")
+    (effects (font (size 1.000759 1.000759) (thickness 0.25019)))
+  )
   (gr_text "PT1000" (at 134.62 56.007 180) (layer "F.SilkS")
     (effects (font (size 1.000759 1.000759) (thickness 0.14986)))
@@
     (effects (font (size 1.000759 1.000759) (thickness 0.14986)))
   )
+  (gr_text "ZIO\nConnector" (at 148.61 95.53) (layer "F.SilkS")
+    (effects (font (size 1.000759 1.000759) (thickness 0.25019)))
+  )
   (gr_text "+      -" (at 72.39 99.06 270) (layer "F.SilkS")
     (effects (font (size 1.000759 1.000759) (thickness 0.14986)))
@@
     (effects (font (size 1.000759 1.000759) (thickness 0.14986)))
   )
+  (gr_text "Morpho" (at 156.09 76.14) (layer "F.SilkS")
+    (effects (font (size 1.000759 1.000759) (thickness 0.25019)))
+  )
   (gr_text "ETH" (at 116.205 78.105) (layer "Eco1.User")
