File: HW_Temperature_Sensors_Board/Espansione_NucleoH723ZG/Kicad_pj/connectors.kicad_sch (KiCad schematic)
At the start: 25 parts, among them CN1 CN11, CN2 CN8, CN3 CN9, CN4 CN7, CN5 CN10, CN6 C12, J3 691382000008, J4 Conn_01x06, J5 Conn_01x02, J6 Screw_Terminal_01x02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

Commit message: hw: connectors update
Other:
- note added: "Morpho"
- note added: "ZIO"
- moved on the sheet: J3
Changed lines of the file:
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@@
     (stroke (width 0) (type default) (color 0 0 0 0))
   )
-  (wire (pts (xy 44.45 176.53) (xy 60.96 176.53))
+  (wire (pts (xy 80.01 186.69) (xy 96.52 186.69))
     (stroke (width 0) (type default) (color 0 0 0 0))
   )
@@
     (stroke (width 0) (type default) (color 0 0 0 0))
   )
-  (wire (pts (xy 44.45 161.29) (xy 60.96 161.29))
+  (wire (pts (xy 80.01 171.45) (xy 96.52 171.45))
     (stroke (width 0) (type default) (color 0 0 0 0))
   )
@@
     (stroke (width 0) (type default) (color 0 0 0 0))
   )
-  (wire (pts (xy 44.45 171.45) (xy 60.96 171.45))
+  (wire (pts (xy 80.01 181.61) (xy 96.52 181.61))
     (stroke (width 0) (type default) (color 0 0 0 0))
   )
@@
     (stroke (width 0) (type default) (color 0 0 0 0))
   )
-  (wire (pts (xy 44.45 173.99) (xy 60.96 173.99))
+  (wire (pts (xy 80.01 184.15) (xy 96.52 184.15))
     (stroke (width 0) (type default) (color 0 0 0 0))
   )
@@
     (stroke (width 0) (type default) (color 0 0 0 0))
   )
-  (wire (pts (xy 44.45 166.37) (xy 60.96 166.37))
+  (wire (pts (xy 80.01 176.53) (xy 96.52 176.53))
     (stroke (width 0) (type default) (color 0 0 0 0))
   )
@@
     (stroke (width 0) (type default) (color 0 0 0 0))
   )
-  (wire (pts (xy 44.45 168.91) (xy 60.96 168.91))
+  (wire (pts (xy 80.01 179.07) (xy 96.52 179.07))
     (stroke (width 0) (type default) (color 0 0 0 0))
   )
@@
     (stroke (width 0) (type default) (color 0 0 0 0))
   )
-  (wire (pts (xy 44.45 179.07) (xy 60.96 179.07))
+  (wire (pts (xy 80.01 189.23) (xy 96.52 189.23))
     (stroke (width 0) (type default) (color 0 0 0 0))
   )
@@
     (stroke (width 0) (type default) (color 0 0 0 0))
   )
-  (wire (pts (xy 44.45 163.83) (xy 60.96 163.83))
+  (wire (pts (xy 80.01 173.99) (xy 96.52 173.99))
     (stroke (width 0) (type default) (color 0 0 0 0))
   )
@@
     (effects (font (size 1 1)) (justify left bottom))
   )
+  (text "Morpho" (at 25.4 34.29 0)
+    (effects (font (size 1.27 1.27) (thickness 0.254) bold italic) (justify left bottom))
+  )
   (text "MOSI_not_used" (at 86.36 97.79 0)
     (effects (font (size 1 1)) (justify left bottom))
@@
     (effects (font (size 1 1)) (justify left bottom))
   )
+  (text "Morpho" (at 140.97 33.02 0)
+    (effects (font (size 1.27 1.27) (thickness 0.254) bold italic) (justify left bottom))
+  )
   (text "PWSTP_MOSI" (at 124.46 57.15 0)
     (effects (font (size 1 1)) (justify left bottom))
   )
+  (text "ZIO\n" (at 55.88 34.29 0)
+    (effects (font (size 1.27 1.27) (thickness 0.254) bold italic) (justify left bottom))
+  )
   (text "PWSTP_MISO" (at 124.46 54.61 0)
     (effects (font (size 1 1)) (justify left bottom))
@@
     (effects (font (size 1.27 1.27)) (justify left bottom))
   )
+  (text "ZIO\n" (at 115.57 34.29 0)
+    (effects (font (size 1.27 1.27) (thickness 0.254) bold italic) (justify left bottom))
+  )
   (text "PWSTP_STCK" (at 124.46 62.23 0)
     (effects (font (size 1 1)) (justify left bottom))
@@
     (effects (font (size 1.27 1.27)) (justify right bottom))
   )
-  (label "ENC_GND" (at 60.96 161.29 0)
+  (label "ENC_GND" (at 96.52 171.45 0)
     (effects (font (size 1.27 1.27)) (justify left bottom))
   )
@@
     (effects (font (size 1.27 1.27)) (justify right bottom))
   )
-  (label "ENC_VCC" (at 55.88 163.83 180)
+  (label "ENC_VCC" (at 91.44 173.99 180)
     (effects (font (size 1.27 1.27)) (justify right bottom))
   )
@@
     (effects (font (size 1.27 1.27)) (justify left))
   )
-  (hierarchical_label "ENC_SSI_DATA-" (shape input) (at 60.96 173.99 0)
+  (hierarchical_label "ENC_SSI_DATA-" (shape input) (at 96.52 184.15 0)
     (effects (font (size 1.27 1.27)) (justify left))
   )
@@
     (effects (font (size 1.27 1.27)) (justify left))
   )
-  (hierarchical_label "ENC_SSI_CLK+" (shape input) (at 60.96 166.37 0)
+  (hierarchical_label "ENC_SSI_CLK+" (shape input) (at 96.52 176.53 0)
     (effects (font (size 1.27 1.27)) (justify left))
   )
@@
     (effects (font (size 1.27 1.27)) (justify left))
   )
-  (hierarchical_label "ENC_SSI_CLK-" (shape input) (at 60.96 168.91 0)
-    (effects (font (size 1.27 1.27)) (justify left))
-  )
-  (hierarchical_label "ENC_VCC" (shape input) (at 60.96 163.83 0)
-    (effects (font (size 1.27 1.27)) (justify left))
-  )
-  (hierarchical_label "ENC_SSI_DATA+" (shape input) (at 60.96 171.45 0)
+  (hierarchical_label "ENC_SSI_CLK-" (shape input) (at 96.52 179.07 0)
+    (effects (font (size 1.27 1.27)) (justify left))
+  )
+  (hierarchical_label "ENC_VCC" (shape input) (at 96.52 173.99 0)
+    (effects (font (size 1.27 1.27)) (justify left))
+  )
+  (hierarchical_label "ENC_SSI_DATA+" (shape input) (at 96.52 181.61 0)
     (effects (font (size 1.27 1.27)) (justify left))
   )
@@
     (effects (font (size 1.27 1.27)) (justify right))
   )
-  (hierarchical_label "ENC_SSI_CLK-" (shape input) (at 60.96 168.91 0)
-    (effects (font (size 1.27 1.27)) (justify left))
-  )
-  (hierarchical_label "ENC_PRESET" (shape input) (at 60.96 176.53 0)
-    (effects (font (size 1.27 1.27)) (justify left))
-  )
-  (hierarchical_label "ENC_DIR" (shape input) (at 60.96 179.07 0)
+  (hierarchical_label "ENC_SSI_CLK-" (shape input) (at 96.52 179.07 0)
+    (effects (font (size 1.27 1.27)) (justify left))
+  )
+  (hierarchical_label "ENC_PRESET" (shape input) (at 96.52 186.69 0)
+    (effects (font (size 1.27 1.27)) (justify left))
+  )
+  (hierarchical_label "ENC_DIR" (shape input) (at 96.52 189.23 0)
     (effects (font (size 1.27 1.27)) (justify left))
   )
@@
     (pin "1")
   )
-  (symbol (lib_id "SamacSys_Parts:691382000008") (at 44.45 161.29 0) (mirror y) (unit 1)
-    (in_bom yes) (on_board yes)
-    (property "Reference" "J3" (id 0) (at 37.0332 154.559 0))
-    (property "Value" "691382000008" (id 1) (at 37.0332 156.8704 0))
-    (property "Footprint" "SamacSys_Parts:SHDR8W80P0X250_1X8_2200X810X1010P" (id 2) (at 27.94 158.75 0)
+  (symbol (lib_id "SamacSys_Parts:691382000008") (at 80.01 171.45 0) (mirror y) (unit 1)
+    (in_bom yes) (on_board yes)
+    (property "Reference" "J3" (id 0) (at 72.5932 164.719 0))
+    (property "Value" "691382000008" (id 1) (at 72.5932 167.0304 0))
+    (property "Footprint" "SamacSys_Parts:SHDR8W80P0X250_1X8_2200X810X1010P" (id 2) (at 63.5 168.91 0)
       (effects (font (size 1.27 1.27)) (justify left) hide)
     )
-    (property "Datasheet" "http://katalog.we-online.de/em/datasheet/6913820000xx.pdf" (id 3) (at 27.94 161.29 0)
+    (property "Datasheet" "http://katalog.we-online.de/em/datasheet/6913820000xx.pdf" (id 3) (at 63.5 171.45 0)
       (effects (font (size 1.27 1.27)) (justify left) hide)
     )
-    (property "Description" "Wurth Elektronik 382 Series 2.5mm Pitch Vertical Pluggable Terminal Block, PCB Header with Solder Termination, 8 Way" (id 4) (at 27.94 163.83 0)
+    (property "Description" "Wurth Elektronik 382 Series 2.5mm Pitch Vertical Pluggable Terminal Block, PCB Header with Solder Termination, 8 Way" (id 4) (at 63.5 173.99 0)
       (effects (font (size 1.27 1.27)) (justify left) hide)
     )
-    (property "Height" "10.1" (id 5) (at 27.94 166.37 0)
+    (property "Height" "10.1" (id 5) (at 63.5 176.53 0)
       (effects (font (size 1.27 1.27)) (justify left) hide)
     )
-    (property "Manufacturer_Name" "Wurth Elektronik" (id 6) (at 27.94 168.91 0)
+    (property "Manufacturer_Name" "Wurth Elektronik" (id 6) (at 63.5 179.07 0)
       (effects (font (size 1.27 1.27)) (justify left) hide)
     )
-    (property "Manufacturer_Part_Number" "691382000008" (id 7) (at 27.94 171.45 0)
+    (property "Manufacturer_Part_Number" "691382000008" (id 7) (at 63.5 181.61 0)
       (effects (font (size 1.27 1.27)) (justify left) hide)
     )
-    (property "Mouser Part Number" "710-691382000008" (id 8) (at 27.94 173.99 0)
+    (property "Mouser Part Number" "710-691382000008" (id 8) (at 63.5 184.15 0)
       (effects (font (size 1.27 1.27)) (justify left) hide)
     )
-    (property "Mouser Price/Stock" "https://www.mouser.co.uk/ProductDetail/Wurth-Elektronik/691382000008?qs=a9WhcLg8qCyuKMyFRlGfoA%3D%3D" (id 9) (at 27.94 176.53 0)
+    (property "Mouser Price/Stock" "https://www.mouser.co.uk/ProductDetail/Wurth-Elektronik/691382000008?qs=a9WhcLg8qCyuKMyFRlGfoA%3D%3D" (id 9) (at 63.5 186.69 0)
       (effects (font (size 1.27 1.27)) (justify left) hide)
     )
-    (property "Arrow Part Number" "" (id 10) (at 27.94 179.07 0)
+    (property "Arrow Part Number" "" (id 10) (at 63.5 189.23 0)
       (effects (font (size 1.27 1.27)) (justify left) hide)
     )
-    (property "Arrow Price/Stock" "" (id 11) (at 27.94 181.61 0)
+    (property "Arrow Price/Stock" "" (id 11) (at 63.5 191.77 0)
       (effects (font (size 1.27 1.27)) (justify left) hide)
     )
